File: pcb/sizif512-wifi.sch (KiCad schematic (older format))
At the start: 13 parts, among them J1 Conn_01x10, U1 AMS1117-3.3, U2 ESP-12E

Commit message: import rev B files
Parts:
- removed R2, R5: 10k, Capacitor_SMD:C_0805_2012Metric_Pad1.15x1.40mm_HandSolder, symbol Device:R
- C2: footprint Capacitor_SMD:C_2010_5025Metric_Pad1.52x2.65mm_HandSolder -> Capacitor_Tantalum_SMD:CP_EIA-6032-15_Kemet-U_Pad2.25x2.35mm_HandSolder
- R1: value 560 -> 47
- U2: footprint ESP8266:ESP-12E_SMD -> RF_Module:ESP-12E
Connections:
- net GND: now also U2.16 (GPIO15)
- net at R6.1, TP1.1, U2.1 (~RST): now also U2.3 (EN)

Commit message: import rev C files
Parts:
- R3, R4: value 560 -> 470
- TP1: footprint Connector_Pin:Pin_D0.7mm_L6.5mm_W1.8mm_FlatFork -> Connector_Pin:Pin_D0.9mm_L10.0mm_W2.4mm_FlatFork
- renumbered R6 to R5
Other:
- moved on the sheet: C1, C2, C3, R1, R3, R4, R5, U1, U2
